Commit message: Add Vulcano macro for composing in project-specific description packages

File: vulcano_description/robots/vulcano_robot.urdf.xacro (robot description, xacro)
@@ -1,57 +1,5 @@
 <?xml version="1.0"?>
 <robot name="vulcano" xmlns:xacro="http://www.ros.org/wiki/xacro">
-  <xacro:property name="PI" value="3.1415926535897931"/>
-  <xacro:arg name="joint_limited" default="false"/>
-  <!-- ***************** -->
-  <!-- Imported elements -->
-  <!-- ***************** -->
-  <!-- First we import all posible elements defined in the urdf.xacro files. All these elements are defined as macro:xacros -->
-  <!-- Import vulcano base -->
-  <xacro:include filename="$(find vulcano_base_description)/urdf/vulcano_base.urdf.xacro" />
-  <!-- Import vulcano torso -->
-  <xacro:include filename="$(find vulcano_torso_description)/urdf/vulcano_torso.urdf.xacro"/>
-  <!-- Import UR10 -->
-  <xacro:include filename="$(find ur_description)/urdf/ur10.urdf.xacro"/>
-  <!--<xacro:include filename="$(find ur_description)/urdf/common.gazebo.xacro"/>-->
-  <!-- Import calibrated UR10 -->
-  <xacro:include filename="$(find vulcano_calibrated_ur_description)/urdf/calibrated_ur10_vulcano_left_arm.urdf.xacro"/>
-  <xacro:include filename="$(find vulcano_calibrated_ur_description)/urdf/calibrated_ur10_vulcano_right_arm.urdf.xacro"/>
-  <!-- Import common gazebo elements -->
-  <xacro:include filename="$(find vulcano_description)/robots/common.gazebo.xacro" />
-  <xacro:property name="hq" value="true" />
-  <xacro:property name="publish_bf" value="true" />
-  <xacro:vulcano_base prefix="" publish_bf="${publish_bf}" hq="${hq}"/>
-  <!-- Fix torso to base -->
-  <joint name="base_torso_joint" type="fixed">
-    <origin xyz="0.47 0.0 0.474" rpy="0.0 0.0 0.0"/>
-    <parent link="base_link"/>
-    <child link="torso_base_link"/>
-    <axis xyz="0 0 0"/>
-  </joint>
-  <xacro:vulcano_torso prefix="" hq="${hq}" />
-  <!-- Fix right arm to torso -->
-  <joint name="torso_right_arm_base_joint" type="fixed">
-    <origin xyz="-0.1622 0.275533 0.021967" rpy="0 ${-PI/4.0} ${-PI/2.0}"/>  <!-- TODO: set correct orientation -->
-    <parent link="torso_tkd668_link"/>
-    <child link="right_arm_base_link"/>
-  </joint>
-  <!--xacro:ur10_robot prefix="right_arm_" joint_limited="$(arg joint_limited)"/-->
-  <xacro:right_arm_ur10_robot prefix="right_arm_" joint_limited="$(arg joint_limited)"/>
-  <!-- Fix left arm to torso -->
-  <joint name="torso_left_arm_base_joint" type="fixed">
-    <origin xyz="-0.1622 -0.275533 0.021967" rpy="0 ${PI/4.0} ${-PI/2.0}"/>
-    <parent link="torso_tkd668_link"/>
-    <child link="left_arm_base_link"/>
-  </joint>
-  <!--xacro:ur10_robot prefix="left_arm_" joint_limited="$(arg joint_limited)"/-->
-  <xacro:left_arm_ur10_robot prefix="left_arm_" joint_limited="$(arg joint_limited)"/>
-  <xacro:tube_support prefix="left_arm_ee_" parent="left_arm_ee_link">
-    <origin xyz="0.012 0 0.0975" rpy="0 0 0"/>
-    <box size="0.075 0.075 0.075" />
-  </xacro:tube_support>
-  <xacro:tube_support prefix="right_arm_ee_" parent="right_arm_ee_link">
-    <origin xyz="0.012 0 0.0975" rpy="0 0 0"/>
-    <box size="0.075 0.075 0.075" />
-  </xacro:tube_support>
-  <xacro:ros_control />
+  <xacro:include filename="$(find vulcano_description)/robots/vulcano.urdf.xacro"/>
+  <xacro:vulcano/>
 </robot>

Commit message: Add Vulcano macro to facilitate composing project-specific URDF models

File: vulcano_description/robots/vulcano_robot.urdf.xacro (robot description, xacro)
@@ -1,77 +1,7 @@
 <?xml version="1.0"?>
 <robot name="vulcano" xmlns:xacro="http://www.ros.org/wiki/xacro">
-  <xacro:property name="PI" value="3.1415926535897931"/>
   <xacro:arg name="joint_limited" default="false"/>
   <xacro:arg name="custom_limits" default="false"/>
-  <!-- ***************** -->
-  <!-- Imported elements -->
-  <!-- ***************** -->
-  <!-- First we import all posible elements defined in the urdf.xacro files. All these elements are defined as macro:xacros -->
-  <!-- Import vulcano base -->
-  <xacro:include filename="$(find vulcano_base_description)/urdf/vulcano_base.urdf.xacro" />
-  <!-- Import vulcano torso -->
-  <xacro:include filename="$(find vulcano_torso_description)/urdf/vulcano_torso.urdf.xacro"/>
-  <!-- Import UR10 -->
-  <xacro:include filename="$(find ur_description)/urdf/ur10.urdf.xacro"/>
-  <!-- Import calibrated UR10 -->
-  <xacro:include filename="$(find vulcano_calibrated_ur_description)/urdf/calibrated_ur10_vulcano_left_arm.urdf.xacro"/>
-  <xacro:include filename="$(find vulcano_calibrated_ur_description)/urdf/calibrated_ur10_vulcano_right_arm.urdf.xacro"/>
-  <!-- Import common gazebo elements -->
-  <xacro:include filename="$(find vulcano_description)/robots/common.gazebo.xacro" />
-  <xacro:property name="hq" value="true" />
-  <xacro:property name="publish_bf" value="true" />
-  <xacro:vulcano_base prefix="" publish_bf="${publish_bf}" hq="${hq}"/>
-  <!-- Fix torso to base -->
-  <joint name="base_torso_joint" type="fixed">
-    <origin xyz="0.47 0.0 0.474" rpy="0.0 0.0 0.0"/>
-    <parent link="base_link"/>
-    <child link="torso_base_link"/>
-    <axis xyz="0 0 0"/>
-  </joint>
-  <xacro:vulcano_torso prefix="" hq="${hq}" />
-  <!-- Fix right arm to torso -->
-  <joint name="torso_right_arm_base_joint" type="fixed">
-    <origin xyz="-0.1622 0.275533 0.021967" rpy="0 ${-PI/4.0} ${-PI/2.0}"/>  <!-- TODO: set correct orientation -->
-    <parent link="torso_tkd668_link"/>
-    <child link="right_arm_base_link"/>
-  </joint>
-  <xacro:if value="$(arg custom_limits)">
-    <xacro:right_arm_ur10_robot prefix="right_arm_" joint_limited="$(arg joint_limited)"
-      shoulder_pan_lower_limit="${0}" shoulder_pan_upper_limit="${pi}"
-      shoulder_lift_lower_limit="${-5*pi/4}" shoulder_lift_upper_limit="${-pi/4}"
-      elbow_joint_lower_limit="${-3*pi/4}" elbow_joint_upper_limit="${pi/4}"
-      wrist_1_lower_limit="${-pi}" wrist_1_upper_limit="${0}"
-      wrist_2_lower_limit="${-pi}" wrist_2_upper_limit="${pi}"
-      wrist_3_lower_limit="${-pi}" wrist_3_upper_limit="${pi}"/>
-  </xacro:if>
-  <xacro:unless value="$(arg custom_limits)">
-    <xacro:right_arm_ur10_robot prefix="right_arm_" joint_limited="$(arg joint_limited)"/>
-  </xacro:unless>
-  <!-- Fix left arm to torso -->
-  <joint name="torso_left_arm_base_joint" type="fixed">
-    <origin xyz="-0.1622 -0.275533 0.021967" rpy="0 ${PI/4.0} ${-PI/2.0}"/>
-    <parent link="torso_tkd668_link"/>
-    <child link="left_arm_base_link"/>
-  </joint>
-  <xacro:if value="$(arg custom_limits)">
-    <xacro:left_arm_ur10_robot prefix="left_arm_" joint_limited="$(arg joint_limited)"
-      shoulder_pan_lower_limit="${-pi}" shoulder_pan_upper_limit="${0}"
-      shoulder_lift_lower_limit="${-3*pi/4}" shoulder_lift_upper_limit="${pi/4}"
-      elbow_joint_lower_limit="${-pi/4}" elbow_joint_upper_limit="${3*pi/4}"
-      wrist_1_lower_limit="${-pi}" wrist_1_upper_limit="${0}"
-      wrist_2_lower_limit="${-pi}" wrist_2_upper_limit="${pi}"
-      wrist_3_lower_limit="${-pi}" wrist_3_upper_limit="${pi}"/>
-  </xacro:if>
-  <xacro:unless value="$(arg custom_limits)">
-    <xacro:left_arm_ur10_robot prefix="left_arm_" joint_limited="$(arg joint_limited)"/>
-  </xacro:unless>
-  <xacro:tube_support prefix="left_arm_ee_" parent="left_arm_ee_link">
-    <origin xyz="0.012 0 0.0975" rpy="0 0 0"/>
-    <box size="0.075 0.075 0.075" />
-  </xacro:tube_support>
-  <xacro:tube_support prefix="right_arm_ee_" parent="right_arm_ee_link">
-    <origin xyz="0.012 0 0.0975" rpy="0 0 0"/>
-    <box size="0.075 0.075 0.075" />
-  </xacro:tube_support>
-  <xacro:ros_control />
+  <xacro:include filename="$(find vulcano_description)/robots/vulcano.urdf.xacro"/>
+  <xacro:vulcano joint_limited="$(arg joint_limited)" custom_limits="$(arg custom_limits)"/>
 </robot>
