Commit message: Expose argument to select UR hardware interface for simulation

File: vulcano_calibrated_ur_description/urdf/calibrated_ur10_vulcano_left_arm.urdf.xacro (robot description, xacro)
@@ -98,5 +98,5 @@
     <xacro:property name="left_arm_wrist_3_joint_c_offset" value="0.00527917" />
     <!--xacro:macro name="left_arm_ur10_robot" params="prefix joint_limited shoulder_pan_lower_limit:=${-pi} shoulder_pan_upper_limit:=${pi} shoulder_lift_lower_limit:=${-pi} shoulder_lift_upper_limit:=${pi} elbow_joint_lower_limit:=${-pi} elbow_joint_upper_limit:=${pi} wrist_1_lower_limit:=${-pi} wrist_1_upper_limit:=${pi} wrist_2_lower_limit:=${-pi} wrist_2_upper_limit:=${pi} wrist_3_lower_limit:=${-pi} wrist_3_upper_limit:=${pi}"-->
-	<xacro:macro name="left_arm_ur10_robot" params="prefix joint_limited shoulder_pan_lower_limit:=${-pi} shoulder_pan_upper_limit:=${pi} shoulder_lift_lower_limit:=${-pi} shoulder_lift_upper_limit:=${pi} elbow_joint_lower_limit:=${-pi} elbow_joint_upper_limit:=${pi} wrist_1_lower_limit:=${-2*pi} wrist_1_upper_limit:=${2*pi} wrist_2_lower_limit:=${-2*pi} wrist_2_upper_limit:=${2*pi} wrist_3_lower_limit:=${-2*pi} wrist_3_upper_limit:=${2*pi}">
+	<xacro:macro name="left_arm_ur10_robot" params="prefix joint_limited shoulder_pan_lower_limit:=${-pi} shoulder_pan_upper_limit:=${pi} shoulder_lift_lower_limit:=${-pi} shoulder_lift_upper_limit:=${pi} elbow_joint_lower_limit:=${-pi} elbow_joint_upper_limit:=${pi} wrist_1_lower_limit:=${-2*pi} wrist_1_upper_limit:=${2*pi} wrist_2_lower_limit:=${-2*pi} wrist_2_upper_limit:=${2*pi} wrist_3_lower_limit:=${-2*pi} wrist_3_upper_limit:=${2*pi} transmission_hw_interface:=hardware_interface/PositionJointInterface">
         <link name="${prefix}base_link">
             <visual>
@@ -454,5 +454,5 @@
             </collision>
         </link>
-        <xacro:ur_arm_transmission prefix="${prefix}" />
+        <xacro:ur_arm_transmission prefix="${prefix}" hw_interface="${transmission_hw_interface}" />
         <xacro:ur_arm_gazebo prefix="${prefix}" />
         <!-- ROS base_link to UR 'Base' Coordinates transform -->

File: vulcano_calibrated_ur_description/urdf/calibrated_ur10_vulcano_right_arm.urdf.xacro (robot description, xacro)
@@ -98,5 +98,5 @@
     <xacro:property name="right_arm_wrist_3_joint_c_offset" value="0.000150637" />
     <!--xacro:macro name="right_arm_ur10_robot" params="prefix joint_limited shoulder_pan_lower_limit:=${-pi} shoulder_pan_upper_limit:=${pi} shoulder_lift_lower_limit:=${-pi} shoulder_lift_upper_limit:=${pi} elbow_joint_lower_limit:=${-pi} elbow_joint_upper_limit:=${pi} wrist_1_lower_limit:=${-pi} wrist_1_upper_limit:=${pi} wrist_2_lower_limit:=${-pi} wrist_2_upper_limit:=${pi} wrist_3_lower_limit:=${-pi} wrist_3_upper_limit:=${pi}"-->
-	<xacro:macro name="right_arm_ur10_robot" params="prefix joint_limited shoulder_pan_lower_limit:=${-pi} shoulder_pan_upper_limit:=${pi} shoulder_lift_lower_limit:=${-pi} shoulder_lift_upper_limit:=${pi} elbow_joint_lower_limit:=${-pi} elbow_joint_upper_limit:=${pi} wrist_1_lower_limit:=${-2*pi} wrist_1_upper_limit:=${2*pi} wrist_2_lower_limit:=${-2*pi} wrist_2_upper_limit:=${2*pi} wrist_3_lower_limit:=${-2*pi} wrist_3_upper_limit:=${2*pi}">
+	<xacro:macro name="right_arm_ur10_robot" params="prefix joint_limited shoulder_pan_lower_limit:=${-pi} shoulder_pan_upper_limit:=${pi} shoulder_lift_lower_limit:=${-pi} shoulder_lift_upper_limit:=${pi} elbow_joint_lower_limit:=${-pi} elbow_joint_upper_limit:=${pi} wrist_1_lower_limit:=${-2*pi} wrist_1_upper_limit:=${2*pi} wrist_2_lower_limit:=${-2*pi} wrist_2_upper_limit:=${2*pi} wrist_3_lower_limit:=${-2*pi} wrist_3_upper_limit:=${2*pi} transmission_hw_interface:=hardware_interface/PositionJointInterface">
         <link name="${prefix}base_link">
             <visual>
@@ -454,5 +454,5 @@
             </collision>
         </link>
-        <xacro:ur_arm_transmission prefix="${prefix}" />
+        <xacro:ur_arm_transmission prefix="${prefix}" hw_interface="${transmission_hw_interface}" />
         <xacro:ur_arm_gazebo prefix="${prefix}" />
         <!-- ROS base_link to UR 'Base' Coordinates transform -->

File: vulcano_description/robots/vulcano.urdf.xacro (robot description, xacro)
@@ -1,5 +1,5 @@
 <?xml version="1.0"?>
 <robot name="vulcano" xmlns:xacro="http://www.ros.org/wiki/xacro">
-  <xacro:macro name="vulcano">
+  <xacro:macro name="vulcano" params="ur_hw_interface:=hardware_interface/PositionJointInterface">
     <xacro:property name="PI" value="3.1415926535897931"/>
     <xacro:arg name="joint_limited" default="false"/>
@@ -38,5 +38,5 @@
     </joint>
     <!--xacro:ur10_robot prefix="right_arm_" joint_limited="$(arg joint_limited)"/-->
-    <xacro:right_arm_ur10_robot prefix="right_arm_" joint_limited="$(arg joint_limited)"/>
+    <xacro:right_arm_ur10_robot prefix="right_arm_" joint_limited="$(arg joint_limited)" transmission_hw_interface="${ur_hw_interface}"/>
     <!-- Fix left arm to torso -->
     <joint name="torso_left_arm_base_joint" type="fixed">
@@ -46,5 +46,5 @@
     </joint>
     <!--xacro:ur10_robot prefix="left_arm_" joint_limited="$(arg joint_limited)"/-->
-    <xacro:left_arm_ur10_robot prefix="left_arm_" joint_limited="$(arg joint_limited)"/>
+    <xacro:left_arm_ur10_robot prefix="left_arm_" joint_limited="$(arg joint_limited)" transmission_hw_interface="${ur_hw_interface}"/>
     <xacro:tube_support prefix="left_arm_ee_" parent="left_arm_ee_link">
       <origin xyz="0.012 0 0.0975" rpy="0 0 0"/>

File: vulcano_description/robots/vulcano_robot.urdf.xacro (robot description, xacro)
@@ -1,5 +1,6 @@
 <?xml version="1.0"?>
 <robot name="vulcano" xmlns:xacro="http://www.ros.org/wiki/xacro">
+  <xacro:arg name="ur_hw_interface" default="hardware_interface/PositionJointInterface"/>
   <xacro:include filename="$(find vulcano_description)/robots/vulcano.urdf.xacro"/>
-  <xacro:vulcano/>
+  <xacro:vulcano ur_hw_interface="$(arg ur_hw_interface)"/>
 </robot>

Commit message: Restore incorrectly deleted macros and delete the duplicates

File: vulcano_calibrated_ur_description/urdf/calibrated_ur10_vulcano_left_arm.urdf.xacro (robot description, xacro)
@@ -98,11 +98,5 @@
     <xacro:property name="left_arm_wrist_3_joint_c_offset" value="0.00527917" />
     <!--xacro:macro name="left_arm_ur10_robot" params="prefix joint_limited shoulder_pan_lower_limit:=${-pi} shoulder_pan_upper_limit:=${pi} shoulder_lift_lower_limit:=${-pi} shoulder_lift_upper_limit:=${pi} elbow_joint_lower_limit:=${-pi} elbow_joint_upper_limit:=${pi} wrist_1_lower_limit:=${-pi} wrist_1_upper_limit:=${pi} wrist_2_lower_limit:=${-pi} wrist_2_upper_limit:=${pi} wrist_3_lower_limit:=${-pi} wrist_3_upper_limit:=${pi}"-->
-	<xacro:macro name="left_arm_ur10_robot" params="prefix joint_limited
-        shoulder_pan_lower_limit:=${-pi} shoulder_pan_upper_limit:=${0}
-        shoulder_lift_lower_limit:=${-3*pi/4} shoulder_lift_upper_limit:=${pi/4}
-        elbow_joint_lower_limit:=${-pi/4} elbow_joint_upper_limit:=${3*pi/4}
-        wrist_1_lower_limit:=${-pi} wrist_1_upper_limit:=${0}
-        wrist_2_lower_limit:=${-pi} wrist_2_upper_limit:=${pi}
-        wrist_3_lower_limit:=${-pi} wrist_3_upper_limit:=${pi}">
+	<xacro:macro name="left_arm_ur10_robot" params="prefix joint_limited shoulder_pan_lower_limit:=${-pi} shoulder_pan_upper_limit:=${pi} shoulder_lift_lower_limit:=${-pi} shoulder_lift_upper_limit:=${pi} elbow_joint_lower_limit:=${-pi} elbow_joint_upper_limit:=${pi} wrist_1_lower_limit:=${-2*pi} wrist_1_upper_limit:=${2*pi} wrist_2_lower_limit:=${-2*pi} wrist_2_upper_limit:=${2*pi} wrist_3_lower_limit:=${-2*pi} wrist_3_upper_limit:=${2*pi}">
         <link name="${prefix}base_link">
             <visual>

File: vulcano_calibrated_ur_description/urdf/calibrated_ur10_vulcano_right_arm.urdf.xacro (robot description, xacro)
@@ -98,11 +98,5 @@
     <xacro:property name="right_arm_wrist_3_joint_c_offset" value="0.000150637" />
     <!--xacro:macro name="right_arm_ur10_robot" params="prefix joint_limited shoulder_pan_lower_limit:=${-pi} shoulder_pan_upper_limit:=${pi} shoulder_lift_lower_limit:=${-pi} shoulder_lift_upper_limit:=${pi} elbow_joint_lower_limit:=${-pi} elbow_joint_upper_limit:=${pi} wrist_1_lower_limit:=${-pi} wrist_1_upper_limit:=${pi} wrist_2_lower_limit:=${-pi} wrist_2_upper_limit:=${pi} wrist_3_lower_limit:=${-pi} wrist_3_upper_limit:=${pi}"-->
-	<xacro:macro name="right_arm_ur10_robot" params="prefix joint_limited
-        shoulder_pan_lower_limit:=${0} shoulder_pan_upper_limit:=${pi}
-        shoulder_lift_lower_limit:=${-5*pi/4} shoulder_lift_upper_limit:=${-pi/4}
-        elbow_joint_lower_limit:=${-3*pi/4} elbow_joint_upper_limit:=${pi/4}
-        wrist_1_lower_limit:=${-pi} wrist_1_upper_limit:=${0}
-        wrist_2_lower_limit:=${-pi} wrist_2_upper_limit:=${pi}
-        wrist_3_lower_limit:=${-pi} wrist_3_upper_limit:=${pi}">
+	<xacro:macro name="right_arm_ur10_robot" params="prefix joint_limited shoulder_pan_lower_limit:=${-pi} shoulder_pan_upper_limit:=${pi} shoulder_lift_lower_limit:=${-pi} shoulder_lift_upper_limit:=${pi} elbow_joint_lower_limit:=${-pi} elbow_joint_upper_limit:=${pi} wrist_1_lower_limit:=${-2*pi} wrist_1_upper_limit:=${2*pi} wrist_2_lower_limit:=${-2*pi} wrist_2_upper_limit:=${2*pi} wrist_3_lower_limit:=${-2*pi} wrist_3_upper_limit:=${2*pi}">
         <link name="${prefix}base_link">
             <visual>

Commit message: Restore (-pi,pi) range for wrist joints in default joint limited version of UR macros

File: vulcano_calibrated_ur_description/urdf/calibrated_ur10_vulcano_left_arm.urdf.xacro (robot description, xacro)
@@ -97,6 +97,5 @@
     <xacro:property name="left_arm_wrist_3_joint_b_offset" value="0.000358152" />
     <xacro:property name="left_arm_wrist_3_joint_c_offset" value="0.00527917" />
-    <!--xacro:macro name="left_arm_ur10_robot" params="prefix joint_limited shoulder_pan_lower_limit:=${-pi} shoulder_pan_upper_limit:=${pi} shoulder_lift_lower_limit:=${-pi} shoulder_lift_upper_limit:=${pi} elbow_joint_lower_limit:=${-pi} elbow_joint_upper_limit:=${pi} wrist_1_lower_limit:=${-pi} wrist_1_upper_limit:=${pi} wrist_2_lower_limit:=${-pi} wrist_2_upper_limit:=${pi} wrist_3_lower_limit:=${-pi} wrist_3_upper_limit:=${pi}"-->
-	<xacro:macro name="left_arm_ur10_robot" params="prefix joint_limited shoulder_pan_lower_limit:=${-pi} shoulder_pan_upper_limit:=${pi} shoulder_lift_lower_limit:=${-pi} shoulder_lift_upper_limit:=${pi} elbow_joint_lower_limit:=${-pi} elbow_joint_upper_limit:=${pi} wrist_1_lower_limit:=${-2*pi} wrist_1_upper_limit:=${2*pi} wrist_2_lower_limit:=${-2*pi} wrist_2_upper_limit:=${2*pi} wrist_3_lower_limit:=${-2*pi} wrist_3_upper_limit:=${2*pi}">
+	<xacro:macro name="left_arm_ur10_robot" params="prefix joint_limited shoulder_pan_lower_limit:=${-pi} shoulder_pan_upper_limit:=${pi} shoulder_lift_lower_limit:=${-pi} shoulder_lift_upper_limit:=${pi} elbow_joint_lower_limit:=${-pi} elbow_joint_upper_limit:=${pi} wrist_1_lower_limit:=${-pi} wrist_1_upper_limit:=${pi} wrist_2_lower_limit:=${-pi} wrist_2_upper_limit:=${pi} wrist_3_lower_limit:=${-pi} wrist_3_upper_limit:=${pi}">
         <link name="${prefix}base_link">
             <visual>

File: vulcano_calibrated_ur_description/urdf/calibrated_ur10_vulcano_right_arm.urdf.xacro (robot description, xacro)
@@ -97,6 +97,5 @@
     <xacro:property name="right_arm_wrist_3_joint_b_offset" value="-0.000202165" />
     <xacro:property name="right_arm_wrist_3_joint_c_offset" value="0.000150637" />
-    <!--xacro:macro name="right_arm_ur10_robot" params="prefix joint_limited shoulder_pan_lower_limit:=${-pi} shoulder_pan_upper_limit:=${pi} shoulder_lift_lower_limit:=${-pi} shoulder_lift_upper_limit:=${pi} elbow_joint_lower_limit:=${-pi} elbow_joint_upper_limit:=${pi} wrist_1_lower_limit:=${-pi} wrist_1_upper_limit:=${pi} wrist_2_lower_limit:=${-pi} wrist_2_upper_limit:=${pi} wrist_3_lower_limit:=${-pi} wrist_3_upper_limit:=${pi}"-->
-	<xacro:macro name="right_arm_ur10_robot" params="prefix joint_limited shoulder_pan_lower_limit:=${-pi} shoulder_pan_upper_limit:=${pi} shoulder_lift_lower_limit:=${-pi} shoulder_lift_upper_limit:=${pi} elbow_joint_lower_limit:=${-pi} elbow_joint_upper_limit:=${pi} wrist_1_lower_limit:=${-2*pi} wrist_1_upper_limit:=${2*pi} wrist_2_lower_limit:=${-2*pi} wrist_2_upper_limit:=${2*pi} wrist_3_lower_limit:=${-2*pi} wrist_3_upper_limit:=${2*pi}">
+	<xacro:macro name="right_arm_ur10_robot" params="prefix joint_limited shoulder_pan_lower_limit:=${-pi} shoulder_pan_upper_limit:=${pi} shoulder_lift_lower_limit:=${-pi} shoulder_lift_upper_limit:=${pi} elbow_joint_lower_limit:=${-pi} elbow_joint_upper_limit:=${pi} wrist_1_lower_limit:=${-pi} wrist_1_upper_limit:=${pi} wrist_2_lower_limit:=${-pi} wrist_2_upper_limit:=${pi} wrist_3_lower_limit:=${-pi} wrist_3_upper_limit:=${pi}">
         <link name="${prefix}base_link">
             <visual>

Commit message: Expose argument to select UR hardware interface for simulation

File: vulcano_calibrated_ur_description/urdf/calibrated_ur10_vulcano_left_arm.urdf.xacro (robot description, xacro)
@@ -97,5 +97,5 @@
     <xacro:property name="left_arm_wrist_3_joint_b_offset" value="0.000358152" />
     <xacro:property name="left_arm_wrist_3_joint_c_offset" value="0.00527917" />
-	<xacro:macro name="left_arm_ur10_robot" params="prefix joint_limited shoulder_pan_lower_limit:=${-pi} shoulder_pan_upper_limit:=${pi} shoulder_lift_lower_limit:=${-pi} shoulder_lift_upper_limit:=${pi} elbow_joint_lower_limit:=${-pi} elbow_joint_upper_limit:=${pi} wrist_1_lower_limit:=${-pi} wrist_1_upper_limit:=${pi} wrist_2_lower_limit:=${-pi} wrist_2_upper_limit:=${pi} wrist_3_lower_limit:=${-pi} wrist_3_upper_limit:=${pi}">
+	<xacro:macro name="left_arm_ur10_robot" params="prefix joint_limited shoulder_pan_lower_limit:=${-pi} shoulder_pan_upper_limit:=${pi} shoulder_lift_lower_limit:=${-pi} shoulder_lift_upper_limit:=${pi} elbow_joint_lower_limit:=${-pi} elbow_joint_upper_limit:=${pi} wrist_1_lower_limit:=${-pi} wrist_1_upper_limit:=${pi} wrist_2_lower_limit:=${-pi} wrist_2_upper_limit:=${pi} wrist_3_lower_limit:=${-pi} wrist_3_upper_limit:=${pi} transmission_hw_interface:=hardware_interface/PositionJointInterface">
         <link name="${prefix}base_link">
             <visual>
@@ -453,5 +453,5 @@
             </collision>
         </link>
-        <xacro:ur_arm_transmission prefix="${prefix}" />
+        <xacro:ur_arm_transmission prefix="${prefix}" hw_interface="${transmission_hw_interface}" />
         <xacro:ur_arm_gazebo prefix="${prefix}" />
         <!-- ROS base_link to UR 'Base' Coordinates transform -->

File: vulcano_calibrated_ur_description/urdf/calibrated_ur10_vulcano_right_arm.urdf.xacro (robot description, xacro)
@@ -97,5 +97,5 @@
     <xacro:property name="right_arm_wrist_3_joint_b_offset" value="-0.000202165" />
     <xacro:property name="right_arm_wrist_3_joint_c_offset" value="0.000150637" />
-	<xacro:macro name="right_arm_ur10_robot" params="prefix joint_limited shoulder_pan_lower_limit:=${-pi} shoulder_pan_upper_limit:=${pi} shoulder_lift_lower_limit:=${-pi} shoulder_lift_upper_limit:=${pi} elbow_joint_lower_limit:=${-pi} elbow_joint_upper_limit:=${pi} wrist_1_lower_limit:=${-pi} wrist_1_upper_limit:=${pi} wrist_2_lower_limit:=${-pi} wrist_2_upper_limit:=${pi} wrist_3_lower_limit:=${-pi} wrist_3_upper_limit:=${pi}">
+	<xacro:macro name="right_arm_ur10_robot" params="prefix joint_limited shoulder_pan_lower_limit:=${-pi} shoulder_pan_upper_limit:=${pi} shoulder_lift_lower_limit:=${-pi} shoulder_lift_upper_limit:=${pi} elbow_joint_lower_limit:=${-pi} elbow_joint_upper_limit:=${pi} wrist_1_lower_limit:=${-pi} wrist_1_upper_limit:=${pi} wrist_2_lower_limit:=${-pi} wrist_2_upper_limit:=${pi} wrist_3_lower_limit:=${-pi} wrist_3_upper_limit:=${pi} transmission_hw_interface:=hardware_interface/PositionJointInterface">
         <link name="${prefix}base_link">
             <visual>
@@ -453,5 +453,5 @@
             </collision>
         </link>
-        <xacro:ur_arm_transmission prefix="${prefix}" />
+        <xacro:ur_arm_transmission prefix="${prefix}" hw_interface="${transmission_hw_interface}" />
         <xacro:ur_arm_gazebo prefix="${prefix}" />
         <!-- ROS base_link to UR 'Base' Coordinates transform -->

File: vulcano_description/robots/vulcano.urdf.xacro (robot description, xacro)
@@ -1,5 +1,5 @@
 <?xml version="1.0"?>
 <robot name="vulcano" xmlns:xacro="http://www.ros.org/wiki/xacro">
-  <xacro:macro name="vulcano" params="joint_limited:=false custom_limits:=false">
+  <xacro:macro name="vulcano" params="joint_limited:=false custom_limits:=false ur_hw_interface:=hardware_interface/PositionJointInterface">
     <xacro:property name="PI" value="3.1415926535897931"/>
     <!-- ***************** -->
@@ -42,8 +42,10 @@
         wrist_1_lower_limit="${-pi}" wrist_1_upper_limit="${0}"
         wrist_2_lower_limit="${-pi}" wrist_2_upper_limit="${pi}"
-        wrist_3_lower_limit="${-pi}" wrist_3_upper_limit="${pi}"/>
+        wrist_3_lower_limit="${-pi}" wrist_3_upper_limit="${pi}"
+        transmission_hw_interface="${ur_hw_interface}"/>
     </xacro:if>
     <xacro:unless value="${custom_limits}">
-      <xacro:right_arm_ur10_robot prefix="right_arm_" joint_limited="${joint_limited}"/>
+      <xacro:right_arm_ur10_robot prefix="right_arm_" joint_limited="${joint_limited}"
+        transmission_hw_interface="${ur_hw_interface}"/>
     </xacro:unless>
     <!-- Fix left arm to torso -->
@@ -60,8 +62,10 @@
         wrist_1_lower_limit="${-pi}" wrist_1_upper_limit="${0}"
         wrist_2_lower_limit="${-pi}" wrist_2_upper_limit="${pi}"
-        wrist_3_lower_limit="${-pi}" wrist_3_upper_limit="${pi}"/>
+        wrist_3_lower_limit="${-pi}" wrist_3_upper_limit="${pi}"
+        transmission_hw_interface="${ur_hw_interface}"/>
     </xacro:if>
     <xacro:unless value="${custom_limits}">
-      <xacro:left_arm_ur10_robot prefix="left_arm_" joint_limited="${joint_limited}"/>
+      <xacro:left_arm_ur10_robot prefix="left_arm_" joint_limited="${joint_limited}"
+        transmission_hw_interface="${ur_hw_interface}"/>
     </xacro:unless>
     <xacro:tube_support prefix="left_arm_ee_" parent="left_arm_ee_link">

File: vulcano_description/robots/vulcano_robot.urdf.xacro (robot description, xacro)
@@ -3,5 +3,6 @@
   <xacro:arg name="joint_limited" default="false"/>
   <xacro:arg name="custom_limits" default="false"/>
+  <xacro:arg name="ur_hw_interface" default="hardware_interface/PositionJointInterface"/>
   <xacro:include filename="$(find vulcano_description)/robots/vulcano.urdf.xacro"/>
-  <xacro:vulcano joint_limited="$(arg joint_limited)" custom_limits="$(arg custom_limits)"/>
+  <xacro:vulcano joint_limited="$(arg joint_limited)" custom_limits="$(arg custom_limits)" ur_hw_interface="$(arg ur_hw_interface)"/>
 </robot>

Commit message: Add parameter for hardware interface in transmission declaration following the UniversalRobot package update

File: vulcano_calibrated_ur_description/urdf/calibrated_ur10_vulcano_left_arm.urdf.xacro (robot description, xacro)
@@ -97,5 +97,5 @@
     <xacro:property name="left_arm_wrist_3_joint_b_offset" value="0.000358152" />
     <xacro:property name="left_arm_wrist_3_joint_c_offset" value="0.00527917" />
-	<xacro:macro name="left_arm_ur10_robot" params="prefix joint_limited shoulder_pan_lower_limit:=${-pi} shoulder_pan_upper_limit:=${pi} shoulder_lift_lower_limit:=${-pi} shoulder_lift_upper_limit:=${pi} elbow_joint_lower_limit:=${-pi} elbow_joint_upper_limit:=${pi} wrist_1_lower_limit:=${-pi} wrist_1_upper_limit:=${pi} wrist_2_lower_limit:=${-pi} wrist_2_upper_limit:=${pi} wrist_3_lower_limit:=${-pi} wrist_3_upper_limit:=${pi}">
+	<xacro:macro name="left_arm_ur10_robot" params="prefix joint_limited shoulder_pan_lower_limit:=${-pi} shoulder_pan_upper_limit:=${pi} shoulder_lift_lower_limit:=${-pi} shoulder_lift_upper_limit:=${pi} elbow_joint_lower_limit:=${-pi} elbow_joint_upper_limit:=${pi} wrist_1_lower_limit:=${-pi} wrist_1_upper_limit:=${pi} wrist_2_lower_limit:=${-pi} wrist_2_upper_limit:=${pi} wrist_3_lower_limit:=${-pi} wrist_3_upper_limit:=${pi} transmission_hw_interface:=hardware_interface/PositionJointInterface">
         <link name="${prefix}base_link">
             <visual>
@@ -453,5 +453,5 @@
             </collision>
         </link>
-        <xacro:ur_arm_transmission prefix="${prefix}" />
+        <xacro:ur_arm_transmission prefix="${prefix}"  hw_interface="${transmission_hw_interface}"/>
         <xacro:ur_arm_gazebo prefix="${prefix}" />
         <!-- ROS base_link to UR 'Base' Coordinates transform -->

File: vulcano_calibrated_ur_description/urdf/calibrated_ur10_vulcano_right_arm.urdf.xacro (robot description, xacro)
@@ -97,5 +97,5 @@
     <xacro:property name="right_arm_wrist_3_joint_b_offset" value="-0.000202165" />
     <xacro:property name="right_arm_wrist_3_joint_c_offset" value="0.000150637" />
-	<xacro:macro name="right_arm_ur10_robot" params="prefix joint_limited shoulder_pan_lower_limit:=${-pi} shoulder_pan_upper_limit:=${pi} shoulder_lift_lower_limit:=${-pi} shoulder_lift_upper_limit:=${pi} elbow_joint_lower_limit:=${-pi} elbow_joint_upper_limit:=${pi} wrist_1_lower_limit:=${-pi} wrist_1_upper_limit:=${pi} wrist_2_lower_limit:=${-pi} wrist_2_upper_limit:=${pi} wrist_3_lower_limit:=${-pi} wrist_3_upper_limit:=${pi}">
+	<xacro:macro name="right_arm_ur10_robot" params="prefix joint_limited shoulder_pan_lower_limit:=${-pi} shoulder_pan_upper_limit:=${pi} shoulder_lift_lower_limit:=${-pi} shoulder_lift_upper_limit:=${pi} elbow_joint_lower_limit:=${-pi} elbow_joint_upper_limit:=${pi} wrist_1_lower_limit:=${-pi} wrist_1_upper_limit:=${pi} wrist_2_lower_limit:=${-pi} wrist_2_upper_limit:=${pi} wrist_3_lower_limit:=${-pi} wrist_3_upper_limit:=${pi} transmission_hw_interface:=hardware_interface/PositionJointInterface">
         <link name="${prefix}base_link">
             <visual>
@@ -453,5 +453,5 @@
             </collision>
         </link>
-        <xacro:ur_arm_transmission prefix="${prefix}" />
+        <xacro:ur_arm_transmission prefix="${prefix}"  hw_interface="${transmission_hw_interface}"/>
         <xacro:ur_arm_gazebo prefix="${prefix}" />
         <!-- ROS base_link to UR 'Base' Coordinates transform -->
